File: H00R1-H/Design/H00R1-H.sch (EAGLE design)
At the start: 1 part, among them P1 HEXABIT_17.32_TOP_HALF

Commit message: -Standarize the files names - Fix some Schematic issues
Other:
- note added: "H00R1-H"
- note added: "H00R1-H_Frontend"
- note removed: "0"
- note removed: "H00R10-H"
- note removed: "H00R10-H_Frontend"
